File: Schematic/KiCad Project/Schematic.sch (KiCad schematic (older format))
At the start: 35 parts, among them M1 Motor_DC, M2 Motor_DC, SW1 SW, U1 L7805

Commit message: 센서 5조 수정
Parts:
- added D?: LED, symbol Device:LED
- added D?: SI5312-H, symbol Device:LED
- added D?: ST5811, symbol Device:D_Photo
- added R?: 330, symbol Device:R_US
- added R?: 220, symbol Device:R_US
- added R?: 1M, symbol Device:R_US
Connections:
- net +5V: now also D?.2 (A), R?.2
- net GND: now also D?.1 (K), D?.1 (K), R?.1
- net LED4: now reaches A1.~ (VIN)
- net LED4: now also R?.2
- new net: D?.2 (A), R?.1 (x2)
- new net ADC4: A1.~ (VIN), D?.1 (K), R?.2
- no-connect marks 14 -> 12
Other:
- moved on the sheet: D1, D10, D11, D12, D13, D2, D3, D4, R1, R10, R11, R12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
